File: Motherboard.brd (EAGLE design)
At the start: 100 x 150 mm, 11 parts

Commit message: add-filets
Parts:
- moved ALTIMETER2 6.00 mm to (35.0, 112.7)
- moved ARDUINO_NANO1 6.00 mm to (45.3, 93.2)
- moved GPS2 6.00 mm to (59.4, 136.1)
- moved IMU 6.00 mm to (43.9, 112.2)
- moved J1 6.00 mm to (45.0, 75.0)
- moved J2 6.00 mm to (29.0, 77.0)
- moved R_SCL 6.00 mm to (22.4, 125.7)
- moved R_SDA 6.00 mm to (22.4, 128.9)
- moved U$1 6.00 mm to (53.2, 43.5)
- moved U$3 6.00 mm to (29.7, 125.9)
- moved U$4 6.00 mm to (29.7, 146.2)
Other:
- board size 100 x 150 mm -> 87.5 x 150 mm
