File: Powerboard.sch (EAGLE design)
At the start: 10 parts

Commit message: wip
Parts:
- removed ALTIMETER2: (no value), microbuilder:HEADER-1X570MIL
- removed ARDUINO_NANO1: (no value), ArduinoNanoV30:ARDUINO_NANO
- removed GPS2: (no value), microbuilder:HEADER-1X970MIL
- removed IMU: YOSTLABSIMU, YOST LABS IMU:YOSTLABSIMU
- removed J1: (no value), SparkFun-Connectors:CONN_08X2_HEADER
- removed J2: (no value), SparkFun-Connectors:CONN_023.5MM
- removed R_SCL, R_SDA: (no value), rcl:R-US_R0603
- removed U$3, U$4: MOUNTINGHOLE2.5, microbuilder:MOUNTINGHOLE2.5
- added IN1: (no value), SparkFun:M05PTH
- added OUT1: (no value), SparkFun:M03PTH
- added R_TRIM: (no value), rcl:R-US_R0603
- added U$2, U$6, U$7, U$8: STAND-OFF, SparkFun:STAND-OFF
Connections:
- removed net 3V3: ALTIMETER2.1, ARDUINO_NANO1.3V3, GPS2.1, IMU.VIN, R_SCL.1, R_SDA.1
- removed net RX: ARDUINO_NANO1.D3, GPS2.5
- removed net SCL: ALTIMETER2.4, ARDUINO_NANO1.A5, IMU.SCL, R_SCL.2
- removed net SDA: ALTIMETER2.5, ARDUINO_NANO1.A4, IMU.SDA, R_SDA.2
- removed net TX: ARDUINO_NANO1.D2, GPS2.6
- new net ON/OFF: IN1.3
- new net PGOOD: IN1.1
- new net SEQ: IN1.2
- new net TRIM: OUT1.1, R_TRIM.2
- new net VIN: IN1.5
- new net VOUT: OUT1.3
- net GND: now also IN1.4, OUT1.2, R_TRIM.1; no longer ALTIMETER2.3, ARDUINO_NANO1.GND@1, ARDUINO_NANO1.GND@2, GPS2.7, IMU.GND

Commit message: more
Parts:
- added J1: (no value), SparkFun-Connectors:CONN_023.5MM
- added J2: (no value), SparkFun-Connectors:BATTERY_CONN_DEANS
Changed lines of the file:
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@@
 <layer number="112" name="tSilk" color="7" fill="1" visible="yes" active="yes"/>
 <layer number="113" name="ReferenceLS" color="7" fill="1" visible="no" active="no"/>
+<layer number="114" name="Badge_Outline" color="7" fill="1" visible="no" active="no"/>
+<layer number="115" name="ReferenceISLANDS" color="7" fill="1" visible="no" active="no"/>
 <layer number="116" name="Patch_BOT" color="9" fill="4" visible="yes" active="yes"/>
 <layer number="118" name="Rect_Pads" color="7" fill="1" visible="no" active="no"/>
@@
 <part name="U$8" library="SparkFun" deviceset="STAND-OFF" device=""/>
 <part name="R_TRIM" library="rcl" library_urn="urn:adsk.eagle:library:334" deviceset="R-US_" device="R0603" package3d_urn="urn:adsk.eagle:package:23555/2"/>
+<part name="J1" library="SparkFun-Connectors" deviceset="CONN_02" device="3.5MM"/>
+<part name="J2" library="SparkFun-Connectors" deviceset="BATTERY_CONN" device="_DEANS"/>
 </parts>
 <sheets>
@@
 <attribute name="VALUE" x="148.59" y="-19.558" size="1.778" layer="96" rot="R180"/>
 </instance>
+<instance part="J1" gate="G$1" x="53.34" y="-35.56" smashed="yes">
+<attribute name="VALUE" x="50.8" y="-40.386" size="1.778" layer="96" font="vector"/>
+<attribute name="NAME" x="50.8" y="-29.972" size="1.778" layer="95" font="vector"/>
+</instance>
+<instance part="J2" gate="G$1" x="53.34" y="-55.88" smashed="yes">
+<attribute name="VALUE" x="50.8" y="-63.5" size="1.778" layer="96" font="vector"/>
+<attribute name="NAME" x="50.8" y="-52.578" size="1.778" layer="95" font="vector"/>
+</instance>
 </instances>

Commit message: routing powerboard
Connections:
- net GND: now also J1.2, J2.-
- net VIN: now also J2.+
- net VOUT: now also J1.1
Other:
- moved on the sheet: J1, J2
Changed lines of the file:
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@@
 <attribute name="VALUE" x="148.59" y="-19.558" size="1.778" layer="96" rot="R180"/>
 </instance>
-<instance part="J1" gate="G$1" x="53.34" y="-35.56" smashed="yes">
-<attribute name="VALUE" x="50.8" y="-40.386" size="1.778" layer="96" font="vector"/>
-<attribute name="NAME" x="50.8" y="-29.972" size="1.778" layer="95" font="vector"/>
+<instance part="J1" gate="G$1" x="175.26" y="-17.78" smashed="yes" rot="R180">
+<attribute name="VALUE" x="177.8" y="-12.954" size="1.778" layer="96" font="vector" rot="R180"/>
+<attribute name="NAME" x="177.8" y="-18.288" size="1.778" layer="95" font="vector" rot="R180"/>
 </instance>
-<instance part="J2" gate="G$1" x="53.34" y="-55.88" smashed="yes">
-<attribute name="VALUE" x="50.8" y="-63.5" size="1.778" layer="96" font="vector"/>
-<attribute name="NAME" x="50.8" y="-52.578" size="1.778" layer="95" font="vector"/>
+<instance part="J2" gate="G$1" x="73.66" y="-40.64" smashed="yes">
+<attribute name="VALUE" x="71.12" y="-48.26" size="1.778" layer="96" font="vector"/>
+<attribute name="NAME" x="71.12" y="-37.338" size="1.778" layer="95" font="vector"/>
 </instance>
 </instances>
@@
 <net name="GND" class="0">
 <segment>
-<wire x1="55.88" y1="-17.78" x2="81.28" y2="-17.78" width="0.1524" layer="91"/>
+<wire x1="55.88" y1="-17.78" x2="91.44" y2="-17.78" width="0.1524" layer="91"/>
 <label x="76.2" y="-17.78" size="1.778" layer="95"/>
 <pinref part="IN1" gate="G$1" pin="4"/>
+<pinref part="J2" gate="G$1" pin="-"/>
+<wire x1="81.28" y1="-43.18" x2="91.44" y2="-40.64" width="0.1524" layer="91"/>
+<wire x1="91.44" y1="-40.64" x2="91.44" y2="-17.78" width="0.1524" layer="91"/>
 </segment>
 <segment>
@@
 <pinref part="R_TRIM" gate="G$1" pin="1"/>
 <wire x1="149.86" y1="-22.86" x2="149.86" y2="-20.32" width="0.1524" layer="91"/>
+<pinref part="J1" gate="G$1" pin="2"/>
+<wire x1="149.86" y1="-20.32" x2="167.64" y2="-20.32" width="0.1524" layer="91"/>
+<junction x="149.86" y="-20.32"/>
 </segment>
 </net>
@@
 <net name="VIN" class="0">
 <segment>
-<wire x1="55.88" y1="-15.24" x2="81.28" y2="-15.24" width="0.1524" layer="91"/>
+<wire x1="55.88" y1="-15.24" x2="88.9" y2="-15.24" width="0.1524" layer="91"/>
 <label x="76.2" y="-15.24" size="1.778" layer="95"/>
 <pinref part="IN1" gate="G$1" pin="5"/>
+<pinref part="J2" gate="G$1" pin="+"/>
+<wire x1="81.28" y1="-40.64" x2="88.9" y2="-38.1" width="0.1524" layer="91"/>
+<wire x1="88.9" y1="-38.1" x2="88.9" y2="-15.24" width="0.1524" layer="91"/>
 </segment>
 </net>
 <net name="VOUT" class="0">
 <segment>
-<wire x1="109.22" y1="-17.78" x2="134.62" y2="-17.78" width="0.1524" layer="91"/>
 <label x="129.54" y="-17.78" size="1.778" layer="95"/>
 <pinref part="OUT1" gate="G$1" pin="3"/>
+<pinref part="J1" gate="G$1" pin="1"/>
+<wire x1="109.22" y1="-17.78" x2="167.64" y2="-17.78" width="0.1524" layer="91"/>
 </segment>
 </net>
