File: Powerboard.brd (EAGLE design)
At the start: 100 x 150 mm, 11 parts

Commit message: wip
Parts:
- removed ALTIMETER2: (no value), microbuilder:1X05_ROUND_70
- removed ARDUINO_NANO1: (no value), ArduinoNanoV30:ARDUINO_NANO
- removed GPS2: (no value), microbuilder:1X09_ROUND_70
- removed IMU: YOSTLABSIMU, YOST LABS IMU:YOSTLABSIMU
- removed J1: (no value), SparkFun-Connectors:2X8
- removed J2: (no value), SparkFun-Connectors:SCREWTERMINAL-3.5MM-2
- removed R_SCL, R_SDA: (no value), rcl:R0603
- removed U$1: (no value), ArduinoNanoV30:RADIO
- removed U$3, U$4: MOUNTINGHOLE2.5, microbuilder:MOUNTINGHOLE_2.5_PLATED
- added IN1: (no value), SparkFun:1X05
- added OUT1: (no value), SparkFun:1X03
- added R_TRIM: (no value), rcl:R0603
- added U$2, U$6, U$7, U$8: STAND-OFF, SparkFun:STAND-OFF
Connections:
- removed net 3V3: ALTIMETER2.1, ARDUINO_NANO1.2, GPS2.1, IMU.VIN, R_SCL.1, R_SDA.1
- removed net 5V: ARDUINO_NANO1.12
- removed net RX: ARDUINO_NANO1.21, GPS2.5
- removed net SCL: ALTIMETER2.4, ARDUINO_NANO1.9, IMU.SCL, R_SCL.2
- removed net SDA: ALTIMETER2.5, ARDUINO_NANO1.8, IMU.SDA, R_SDA.2
- removed net TX: ARDUINO_NANO1.20, GPS2.6
- new net ON/OFF: IN1.3
- new net PGOOD: IN1.1
- new net SEQ: IN1.2
- new net TRIM: OUT1.1, R_TRIM.2
- new net VOUT: OUT1.3
- net GND: now also IN1.4, OUT1.2, R_TRIM.1; no longer ALTIMETER2.3, ARDUINO_NANO1.14, ARDUINO_NANO1.19, GPS2.7, IMU.GND
- net VIN: now also IN1.5; no longer ARDUINO_NANO1.15
Routing:
- added copper zone on layer 1, net GND
- added copper zone on layer 16, net GND
Other:
- board size 100 x 150 mm -> 95 x 150 mm
- board text added: "ON"
- board text added: "PGD"
- board text added: "SEQ"
- board text added: "TRIM"
- board text added: "VOUT"
- board text removed: "3.3V"
- board text removed: "3Vo"
- board text removed: "EN"
- board text removed: "FIX"
- board text removed: "PPS"
- board text removed: "RX"
- board text removed: "SCL"
- board text removed: "SDA"
- board text removed: "TX"
- board text removed: "VBAT"

Commit message: more
Parts:
- added J1: (no value), SparkFun-Connectors:SCREWTERMINAL-3.5MM-2
- added J2: (no value), SparkFun-Connectors:DEANS
- moved R_TRIM 142.9 mm to (49.0, 132.0), turned to 270 degrees
- moved U$2 78.6 mm to (34.9, 145.3), turned to 270 degrees
- moved IN1 70.9 mm to (34.9, 138.9), turned to 270 degrees
- moved U$7 69.2 mm to (57.7, 145.3), turned to 270 degrees
- moved U$6 52.6 mm to (34.9, 122.4), turned to 270 degrees
- moved OUT1 49.5 mm to (57.7, 131.3), turned to 90 degrees
- moved U$8 37.1 mm to (57.7, 122.4), turned to 270 degrees
Routing:
- removed copper zone on layer 1, net GND
- removed copper zone on layer 16, net GND
Other:
- outline, holes or cut-outs redrawn
Changed lines of the file:
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@@
 <layer number="112" name="tSilk" color="7" fill="1" visible="yes" active="yes"/>
 <layer number="113" name="ReferenceLS" color="7" fill="1" visible="no" active="no"/>
+<layer number="114" name="Badge_Outline" color="7" fill="1" visible="no" active="no"/>
+<layer number="115" name="ReferenceISLANDS" color="7" fill="1" visible="no" active="no"/>
 <layer number="116" name="Patch_BOT" color="9" fill="4" visible="yes" active="yes"/>
 <layer number="118" name="Rect_Pads" color="7" fill="1" visible="no" active="no"/>
@@
 <wire x1="95" y1="150" x2="0" y2="150" width="0" layer="20"/>
 <wire x1="0" y1="150" x2="0" y2="0" width="0" layer="20"/>
-<wire x1="10.16" y1="67.31" x2="38.1" y2="67.31" width="0.2032" layer="20"/>
-<wire x1="38.1" y1="67.31" x2="38.1" y2="95.25" width="0.2032" layer="20"/>
-<wire x1="38.1" y1="95.25" x2="10.16" y2="95.25" width="0.2032" layer="20"/>
-<wire x1="10.16" y1="95.25" x2="10.16" y2="67.31" width="0.2032" layer="20"/>
-<text x="29.845" y="71.374" size="1.27" layer="21" font="vector" ratio="15" rot="R90">VIN</text>
-<text x="27.305" y="71.374" size="1.27" layer="21" font="vector" ratio="15" rot="R90">GND</text>
-<text x="19.685" y="71.374" size="1.27" layer="21" font="vector" ratio="15" rot="R90">PGD</text>
-<text x="22.225" y="71.374" size="1.27" layer="21" font="vector" ratio="15" rot="R90">SEQ</text>
-<text x="24.765" y="71.374" size="1.27" layer="21" font="vector" ratio="15" rot="R90">ON</text>
-<text x="23.5966" y="91.313" size="1.016" layer="21" font="vector" ratio="15" rot="R270">GND</text>
-<text x="21.0566" y="91.313" size="1.016" layer="21" font="vector" ratio="15" rot="R270">VOUT</text>
-<text x="26.1366" y="91.313" size="1.016" layer="21" font="vector" ratio="15" rot="R270">TRIM</text>
+<wire x1="32.31" y1="147.84" x2="32.31" y2="119.9" width="0.2032" layer="51"/>
+<wire x1="32.31" y1="119.9" x2="60.25" y2="119.9" width="0.2032" layer="51"/>
+<wire x1="60.25" y1="119.9" x2="60.25" y2="147.84" width="0.2032" layer="51"/>
+<wire x1="60.25" y1="147.84" x2="32.31" y2="147.84" width="0.2032" layer="51"/>
+<text x="36.374" y="128.155" size="1.27" layer="21" font="vector" ratio="15">VIN</text>
+<text x="36.374" y="130.695" size="1.27" layer="21" font="vector" ratio="15">GND</text>
+<text x="36.374" y="138.315" size="1.27" layer="21" font="vector" ratio="15">PGD</text>
+<text x="36.374" y="135.775" size="1.27" layer="21" font="vector" ratio="15">SEQ</text>
+<text x="36.374" y="133.235" size="1.27" layer="21" font="vector" ratio="15">ON</text>
+<text x="56.313" y="134.4034" size="1.016" layer="21" font="vector" ratio="15" rot="R180">GND</text>
+<text x="56.313" y="136.9434" size="1.016" layer="21" font="vector" ratio="15" rot="R180">VOUT</text>
+<text x="56.313" y="131.8634" size="1.016" layer="21" font="vector" ratio="15" rot="R180">TRIM</text>
 </plain>
 <attributes>
@@
 </autorouter>
 <elements>
-<element name="IN1" library="SparkFun" package="1X05" value="" x="19.05" y="69.85" smashed="yes">
-<attribute name="NAME" x="17.7038" y="71.6788" size="1.27" layer="25" ratio="10"/>
-<attribute name="VALUE" x="17.78" y="66.675" size="1.27" layer="27"/>
-</element>
-<element name="OUT1" library="SparkFun" package="1X03" value="" x="26.67" y="92.71" smashed="yes" rot="R180">
-<attribute name="NAME" x="28.0162" y="90.8812" size="1.27" layer="25" ratio="10" rot="R180"/>
-<attribute name="VALUE" x="27.94" y="95.885" size="1.27" layer="27" rot="R180"/>
-</element>
-<element name="U$2" library="SparkFun" package="STAND-OFF" value="STAND-OFF" x="12.7" y="69.85" smashed="yes"/>
-<element name="U$6" library="SparkFun" package="STAND-OFF" value="STAND-OFF" x="35.56" y="69.85" smashed="yes"/>
-<element name="U$7" library="SparkFun" package="STAND-OFF" value="STAND-OFF" x="12.7" y="92.71" smashed="yes"/>
-<element name="U$8" library="SparkFun" package="STAND-OFF" value="STAND-OFF" x="35.56" y="92.71" smashed="yes"/>
-<element name="R_TRIM" library="rcl" library_urn="urn:adsk.eagle:library:334" package="R0603" package3d_urn="urn:adsk.eagle:package:23555/2" value="" x="2" y="-3" smashed="yes">
-<attribute name="NAME" x="1.365" y="-2.365" size="1.27" layer="25"/>
-<attribute name="SPICEPREFIX" value="R" x="2" y="-3" size="1.778" layer="27" display="off"/>
-<attribute name="VALUE" x="1.365" y="-4.905" size="1.27" layer="27"/>
+<element name="IN1" library="SparkFun" package="1X05" value="" x="34.85" y="138.95" smashed="yes" rot="R270">
+<attribute name="NAME" x="36.6788" y="140.2962" size="1.27" layer="25" ratio="10" rot="R270"/>
+<attribute name="VALUE" x="31.675" y="140.22" size="1.27" layer="27" rot="R270"/>
+</element>
+<element name="OUT1" library="SparkFun" package="1X03" value="" x="57.71" y="131.33" smashed="yes" rot="R90">
+<attribute name="NAME" x="55.8812" y="129.9838" size="1.27" layer="25" ratio="10" rot="R90"/>
+<attribute name="VALUE" x="60.885" y="130.06" size="1.27" layer="27" rot="R90"/>
+</element>
+<element name="U$2" library="SparkFun" package="STAND-OFF" value="STAND-OFF" x="34.85" y="145.3" smashed="yes" rot="R270"/>
+<element name="U$6" library="SparkFun" package="STAND-OFF" value="STAND-OFF" x="34.85" y="122.44" smashed="yes" rot="R270"/>
+<element name="U$7" library="SparkFun" package="STAND-OFF" value="STAND-OFF" x="57.71" y="145.3" smashed="yes" rot="R270"/>
+<element name="U$8" library="SparkFun" package="STAND-OFF" value="STAND-OFF" x="57.71" y="122.44" smashed="yes" rot="R270"/>
+<element name="R_TRIM" library="rcl" library_urn="urn:adsk.eagle:library:334" package="R0603" package3d_urn="urn:adsk.eagle:package:23555/2" value="" x="49" y="132" smashed="yes" rot="R270">
+<attribute name="NAME" x="49.635" y="132.635" size="1.27" layer="25" rot="R270"/>
+<attribute name="SPICEPREFIX" value="R" x="49" y="132" size="1.778" layer="27" rot="R270" display="off"/>
+<attribute name="VALUE" x="47.095" y="132.635" size="1.27" layer="27" rot="R270"/>
+</element>
+<element name="J1" library="SparkFun-Connectors" package="SCREWTERMINAL-3.5MM-2" value="" x="66" y="133" smashed="yes" rot="R90">
+<attribute name="NAME" x="63.46" y="131.73" size="0.6096" layer="25" font="vector" ratio="20" rot="R90"/>
+<attribute name="PROD_ID" value="CONN-08399" x="66" y="133" size="1.778" layer="27" rot="R90" display="off"/>
+<attribute name="VALUE" x="64.73" y="131.73" size="0.6096" layer="27" font="vector" ratio="20" rot="R90"/>
+</element>
+<element name="J2" library="SparkFun-Connectors" package="DEANS" value="" x="22" y="136" smashed="yes">
+<attribute name="NAME" x="18.19" y="138.54" size="0.6096" layer="25" font="vector" ratio="20"/>
+<attribute name="SF_ID" value="PRT-11864" x="22" y="136" size="1.778" layer="27" display="off"/>
+<attribute name="VALUE" x="18.698" y="124.189" size="0.6096" layer="27" font="vector" ratio="20"/>
 </element>
 </elements>
@@
 <contactref element="IN1" pad="4"/>
 <contactref element="OUT1" pad="2"/>
-<polygon width="0.2032" layer="1" isolate="0.3048">
-<vertex x="10.16" y="95.25"/>
-<vertex x="38.1" y="95.25"/>
-<vertex x="38.1" y="67.31"/>
-<vertex x="10.16" y="67.31"/>
-</polygon>
-<polygon width="0.2032" layer="16" isolate="0.3048">
-<vertex x="10.16" y="67.31"/>
-<vertex x="38.1" y="67.31"/>
-<vertex x="38.1" y="95.25"/>
-<vertex x="10.16" y="95.25"/>
-</polygon>
 <contactref element="R_TRIM" pad="1"/>
-<wire x1="26.67" y1="69.85" x2="24.13" y2="92.71" width="0" layer="19" extent="1-1"/>
-<wire x1="1.15" y1="-3" x2="26.67" y2="69.85" width="0" layer="19" extent="1-1"/>
+<wire x1="34.85" y1="131.33" x2="57.71" y2="133.87" width="0" layer="19" extent="1-1"/>
+<wire x1="49" y1="132.85" x2="34.85" y2="131.33" width="0" layer="19" extent="1-1"/>
 </signal>
 <signal name="SEQ">
 <contactref element="IN1" pad="2"/>
-<wire x1="21.59" y1="69.85" x2="21.59" y2="69.8754" width="0.254" layer="16"/>
-<wire x1="21.59" y1="69.85" x2="21.66" y2="69.85" width="0.254" layer="16"/>
+<wire x1="34.85" y1="136.41" x2="34.8754" y2="136.41" width="0.254" layer="16"/>
+<wire x1="34.85" y1="136.41" x2="34.85" y2="136.34" width="0.254" layer="16"/>
 </signal>
 <signal name="PGOOD">
@@
 <contactref element="OUT1" pad="1"/>
 <contactref element="R_TRIM" pad="2"/>
-<wire x1="2.85" y1="-3" x2="26.67" y2="92.71" width="0" layer="19" extent="1-1"/>
+<wire x1="49" y1="131.15" x2="57.71" y2="131.33" width="0" layer="19" extent="1-1"/>
 </signal>
 <signal name="ON/OFF">

Commit message: add-filets
Other:
- board size 95 x 150 mm -> 87.5 x 150 mm
Changed lines of the file:
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@@
 <setting verticaltext="up"/>
 </settings>
-<grid distance="1" unitdist="mm" unit="mm" style="dots" multiple="1" display="yes" altdistance="5" altunitdist="mil" altunit="mil"/>
+<grid distance="0.5" unitdist="mm" unit="mm" style="dots" multiple="1" display="yes" altdistance="5" altunitdist="mil" altunit="mil"/>
 <layers>
 <layer number="1" name="Top" color="4" fill="1" visible="yes" active="yes"/>
@@
 <board>
 <plain>
-<wire x1="0" y1="0" x2="95" y2="0" width="0" layer="20"/>
-<wire x1="95" y1="0" x2="95" y2="150" width="0" layer="20"/>
-<wire x1="95" y1="150" x2="0" y2="150" width="0" layer="20"/>
-<wire x1="0" y1="150" x2="0" y2="0" width="0" layer="20"/>
+<wire x1="3" y1="0" x2="84.5" y2="0" width="0" layer="20"/>
+<wire x1="84.5" y1="0" x2="87.5" y2="3" width="0" layer="20" curve="90"/>
+<wire x1="87.5" y1="3" x2="87.5" y2="147" width="0" layer="20"/>
+<wire x1="87.5" y1="147" x2="84.5" y2="150" width="0" layer="20" curve="90"/>
+<wire x1="84.5" y1="150" x2="3" y2="150" width="0" layer="20"/>
+<wire x1="3" y1="150" x2="0" y2="147" width="0" layer="20" curve="90"/>
+<wire x1="0" y1="147" x2="0" y2="3" width="0" layer="20"/>
+<wire x1="0" y1="3" x2="3" y2="0" width="0" layer="20" curve="90"/>
 <wire x1="32.31" y1="147.84" x2="32.31" y2="119.9" width="0.2032" layer="51"/>
 <wire x1="32.31" y1="119.9" x2="60.25" y2="119.9" width="0.2032" layer="51"/>
@@
 <text x="56.313" y="136.9434" size="1.016" layer="21" font="vector" ratio="15" rot="R180">VOUT</text>
 <text x="56.313" y="131.8634" size="1.016" layer="21" font="vector" ratio="15" rot="R180">TRIM</text>
+<hole x="9.75" y="140" drill="5.5"/>
+<hole x="9.75" y="10" drill="5.5"/>
+<hole x="77.75" y="10" drill="5.5"/>
+<hole x="77.75" y="140" drill="5.5"/>
+<dimension x1="77.75" y1="142.75" x2="77.75" y2="137.25" x3="97" y3="140" textsize="1.778" layer="1" dtype="diameter"/>
+<dimension x1="78" y1="140" x2="10" y2="140" x3="44" y3="169" textsize="1.778" layer="1" dtype="diameter"/>
+<dimension x1="10" y1="9" x2="10" y2="139" x3="-10" y3="74" textsize="1.778" layer="1" dtype="diameter"/>
+<dimension x1="26" y1="150" x2="26" y2="0" x3="-15" y3="75" textsize="1.778" layer="1"/>
+<dimension x1="0" y1="49.5" x2="87.5" y2="49.5" x3="43.75" y3="-7" textsize="1.778" layer="1"/>
 </plain>
 <attributes>

Commit message: routing powerboard
Parts:
- moved J2 13.8 mm to (17.5, 123.0), turned to 180 degrees
Connections:
- net GND: now also J1.2, J2.-
- net VIN: now also J2.+
- net VOUT: now also J1.1
Routing:
- added copper zone on layer 1, net GND
- added copper zone on layer 1, net TRIM
- added copper zone on layer 1, net VIN
- added copper zone on layer 1, net VOUT
Other:
- board text added: "+"
- board text added: "-"
- board text added: "Power Board"
- board text added: "uORocketry"
- board text added: "v1.0"
Changed lines of the file:
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@@
 <setting verticaltext="up"/>
 </settings>
-<grid distance="0.5" unitdist="mm" unit="mm" style="dots" multiple="1" display="yes" altdistance="5" altunitdist="mil" altunit="mil"/>
+<grid distance="0.25" unitdist="mm" unit="mm" style="dots" multiple="1" display="yes" altdistance="5" altunitdist="mil" altunit="mil"/>
 <layers>
 <layer number="1" name="Top" color="4" fill="1" visible="yes" active="yes"/>
@@
 <layer number="45" name="Holes" color="7" fill="1" visible="yes" active="yes"/>
 <layer number="46" name="Milling" color="3" fill="1" visible="no" active="yes"/>
-<layer number="47" name="Measures" color="7" fill="1" visible="no" active="yes"/>
+<layer number="47" name="Measures" color="7" fill="1" visible="yes" active="yes"/>
 <layer number="48" name="Document" color="7" fill="1" visible="yes" active="yes"/>
 <layer number="49" name="Reference" color="7" fill="1" visible="yes" active="yes"/>
@@
 <hole x="77.75" y="10" drill="5.5"/>
 <hole x="77.75" y="140" drill="5.5"/>
-<dimension x1="77.75" y1="142.75" x2="77.75" y2="137.25" x3="97" y3="140" textsize="1.778" layer="1" dtype="diameter"/>
-<dimension x1="78" y1="140" x2="10" y2="140" x3="44" y3="169" textsize="1.778" layer="1" dtype="diameter"/>
-<dimension x1="10" y1="9" x2="10" y2="139" x3="-10" y3="74" textsize="1.778" layer="1" dtype="diameter"/>
-<dimension x1="26" y1="150" x2="26" y2="0" x3="-15" y3="75" textsize="1.778" layer="1"/>
-<dimension x1="0" y1="49.5" x2="87.5" y2="49.5" x3="43.75" y3="-7" textsize="1.778" layer="1"/>
+<dimension x1="77.75" y1="142.75" x2="77.75" y2="137.25" x3="97" y3="140" textsize="1.778" layer="47" dtype="diameter"/>
+<dimension x1="78" y1="140" x2="10" y2="140" x3="44" y3="169" textsize="1.778" layer="47" dtype="diameter"/>
+<dimension x1="10" y1="9" x2="10" y2="139" x3="-10" y3="74" textsize="1.778" layer="47" dtype="diameter"/>
+<dimension x1="26" y1="150" x2="26" y2="0" x3="-15" y3="75" textsize="1.778" layer="47"/>
+<dimension x1="0" y1="49.5" x2="87.5" y2="49.5" x3="43.75" y3="-7" textsize="1.778" layer="47"/>
+<text x="70.5" y="132" size="1.778" layer="47">+</text>
+<text x="70.5" y="136" size="1.778" layer="47">-</text>
+<text x="71" y="129" size="1.778" layer="48">uORocketry </text>
+<text x="70.5" y="125.5" size="1.778" layer="48">Power Board</text>
+<text x="74.5" y="122.5" size="1.778" layer="48">v1.0</text>
 </plain>
 <attributes>
@@
 <attribute name="VALUE" x="64.73" y="131.73" size="0.6096" layer="27" font="vector" ratio="20" rot="R90"/>
 </element>
-<element name="J2" library="SparkFun-Connectors" package="DEANS" value="" x="22" y="136" smashed="yes">
-<attribute name="NAME" x="18.19" y="138.54" size="0.6096" layer="25" font="vector" ratio="20"/>
-<attribute name="SF_ID" value="PRT-11864" x="22" y="136" size="1.778" layer="27" display="off"/>
-<attribute name="VALUE" x="18.698" y="124.189" size="0.6096" layer="27" font="vector" ratio="20"/>
+<element name="J2" library="SparkFun-Connectors" package="DEANS" value="" x="17.5" y="123" smashed="yes" rot="R180">
+<attribute name="NAME" x="21.31" y="120.46" size="0.6096" layer="25" font="vector" ratio="20" rot="R180"/>
+<attribute name="SF_ID" value="PRT-11864" x="17.5" y="123" size="1.778" layer="27" rot="R180" display="off"/>
+<attribute name="VALUE" x="20.802" y="134.811" size="0.6096" layer="27" font="vector" ratio="20" rot="R180"/>
 </element>
 </elements>
@@
 <contactref element="OUT1" pad="2"/>
 <contactref element="R_TRIM" pad="1"/>
-<wire x1="34.85" y1="131.33" x2="57.71" y2="133.87" width="0" layer="19" extent="1-1"/>
-<wire x1="49" y1="132.85" x2="34.85" y2="131.33" width="0" layer="19" extent="1-1"/>
+<contactref element="J2" pad="-"/>
+<contactref element="J1" pad="2"/>
+<polygon width="0.1524" layer="1" thermals="no">
+<vertex x="13.5" y="126"/>
+<vertex x="18" y="125.5"/>
+<vertex x="13.5" y="125.5"/>
+</polygon>
+<polygon width="0.1524" layer="1" thermals="no" rank="6">
+<vertex x="0" y="150"/>
+<vertex x="0" y="0"/>
+<vertex x="87.5" y="0"/>
+<vertex x="87.5" y="150"/>
+</polygon>
+<wire x1="34.85" y1="131.33" x2="16.7634" y2="129.9215" width="0" layer="19" extent="1-1"/>
 </signal>
 <signal name="SEQ">
@@
 <contactref element="OUT1" pad="1"/>
 <contactref element="R_TRIM" pad="2"/>
-<wire x1="49" y1="131.15" x2="57.71" y2="131.33" width="0" layer="19" extent="1-1"/>
+<polygon width="0.1524" layer="1" thermals="no">
+<vertex x="48.25" y="131.75"/>
+<vertex x="49.75" y="131.75"/>
+<vertex x="56" y="131.75"/>
+<vertex x="57" y="132.5"/>
+<vertex x="58.5" y="132.5"/>
+<vertex x="59" y="132"/>
+<vertex x="59" y="130.75"/>
+<vertex x="58.25" y="130"/>
+<vertex x="48.25" y="130"/>
+</polygon>
 </signal>
 <signal name="ON/OFF">
@@
 <signal name="VIN">
 <contactref element="IN1" pad="5"/>
+<contactref element="J2" pad="+"/>
+<polygon width="0.1524" layer="1" thermals="no">
+<vertex x="14" y="125"/>
+<vertex x="21.5" y="125"/>
+<vertex x="29" y="125"/>
+<vertex x="33" y="129.5"/>
+<vertex x="36.5" y="129.5"/>
+<vertex x="36.5" y="127"/>
+<vertex x="33" y="127"/>
+<vertex x="28" y="121"/>
+<vertex x="14" y="121"/>
+</polygon>
+<wire x1="34.85" y1="128.79" x2="17.5" y2="123" width="0" layer="19" extent="1-1"/>
 </signal>
 <signal name="VOUT">
 <contactref element="OUT1" pad="3"/>
+<contactref element="J1" pad="1"/>
+<polygon width="0.1524" layer="1" thermals="no">
+<vertex x="56.25" y="135.25"/>
+<vertex x="56.25" y="137.75"/>
+<vertex x="58.25" y="137.75"/>
+<vertex x="62.5" y="134.5"/>
+<vertex x="67.5" y="134.5"/>
+<vertex x="67.5" y="131.5"/>
+<vertex x="63.5" y="131.5"/>
+<vertex x="58.75" y="135.25"/>
+</polygon>
 </signal>
 </signals>

Commit message: keepout
Routing:
- net GND: track 0.00 -> 18.8 mm
Changed lines of the file:
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@@
 <text x="70.5" y="125.5" size="1.778" layer="48">Power Board</text>
 <text x="74.5" y="122.5" size="1.778" layer="48">v1.0</text>
+<circle x="9.75" y="140" radius="4.125" width="0" layer="39"/>
+<circle x="77.75" y="140" radius="4.125" width="0" layer="39"/>
+<circle x="77.75" y="10" radius="4.125" width="0" layer="39"/>
+<circle x="9.75" y="10" radius="4.125" width="0" layer="39"/>
 </plain>
 <attributes>
@@
 <vertex x="87.5" y="150"/>
 </polygon>
-<wire x1="34.85" y1="131.33" x2="16.7634" y2="129.9215" width="0" layer="19" extent="1-1"/>
+<wire x1="16.7634" y1="129.9215" x2="19.251728125" y2="129.8909875" width="8" layer="1"/>
+<wire x1="19.251728125" y1="129.8909875" x2="30.75" y2="129.75" width="0.1524" layer="1"/>
+<wire x1="30.75" y1="129.75" x2="32" y2="131.25" width="0.1524" layer="1"/>
+<wire x1="32" y1="131.25" x2="34.85" y2="131.33" width="0.1524" layer="1"/>
 </signal>
 <signal name="SEQ">

Commit message: powerboard
Routing:
- net VIN: track 0.00 -> 4.75 mm
Changed lines of the file:
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@@
 <polygon width="0.1524" layer="1" thermals="no">
 <vertex x="14" y="125"/>
-<vertex x="21.5" y="125"/>
 <vertex x="29" y="125"/>
-<vertex x="33" y="129.5"/>
-<vertex x="36.5" y="129.5"/>
+<vertex x="33.44444375" y="130"/>
+<vertex x="36.5" y="130"/>
 <vertex x="36.5" y="127"/>
 <vertex x="33" y="127"/>
@@
 <vertex x="14" y="121"/>
 </polygon>
-<wire x1="34.85" y1="128.79" x2="17.5" y2="123" width="0" layer="19" extent="1-1"/>
+<wire x1="17.5" y1="123" x2="22.25" y2="123" width="3.75" layer="1"/>
 </signal>
 <signal name="VOUT">
