File: Motherboard/Motherboard.brd (EAGLE design)
At the start: 87.5 x 150 mm, 11 parts

Commit message: review1
Parts:
- moved POWER_IN 7.00 mm to (12.5, 133.0)
- moved AIR_BRAKE 6.40 mm to (42.5, 17.0)
- moved ARDUINO_NANO1 4.00 mm to (33.8, 88.7)
Connections:
- net SBG_RX: now also ARDUINO_NANO1.27; no longer ARDUINO_NANO1.23
- net SBG_TX: now also ARDUINO_NANO1.26; no longer ARDUINO_NANO1.22
- net SS: now also ARDUINO_NANO1.22; no longer ARDUINO_NANO1.28
Routing:
- net 5V: track 122.9 -> 130.7 mm
- net SCL: track 104.3 -> 108.7 mm
- net RX: track 26.1 -> 22.3 mm
- net RX0: track 38.3 -> 42.1 mm
- net TX1: track 40.1 -> 43.7 mm
- net MISO: track 94.0 -> 90.5 mm
- net +5V: track 165.3 -> 161.9 mm
- net N$4: track 128.4 -> 125.5 mm
- net SCK: track 57.4 -> 60.1 mm
- net MOSI: track 88.8 -> 86.3 mm
- net 3V3: track 113.0 -> 115.3 mm
- net TX: track 25.8 -> 26.7 mm
- net SS: track 86.4 -> 85.9 mm
- net SDA: track 113.1 -> 113.6 mm

Commit message: layout r2
Parts:
- moved U$3 8.75 mm to (26.8, 148.0)
- moved POWER_IN 5.26 mm to (17.8, 132.8)
Routing:
- net GND: track 224.0 -> 0.00 mm
- net +5V: track 161.9 -> 0.00 mm
- net 5V: track 130.7 -> 0.00 mm
- net N$4: track 125.5 -> 0.00 mm
- net 3V3: track 115.3 -> 0.00 mm, vias 2 -> 0
- net SDA: track 113.6 -> 0.00 mm, vias 2 -> 0
- net SCL: track 108.7 -> 0.00 mm, vias 1 -> 0
- net MISO: track 90.5 -> 0.00 mm
- net MOSI: track 86.3 -> 0.00 mm
- net SS: track 85.9 -> 0.00 mm
- net SCK: track 60.1 -> 0.00 mm, vias 1 -> 0
- net SBG_TX: track 53.9 -> 0.00 mm
- net SBG_RX: track 44.0 -> 0.00 mm
- net TX1: track 43.7 -> 0.00 mm, vias 2 -> 0
- net RX0: track 42.1 -> 0.00 mm, vias 1 -> 0
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Other:
- board text added: "+"
- board text added: "-"
- board text added: "AIR BRAKE"
- board text added: "DATA"

Commit message: routed motherboard r2
Routing:
- net GND: track 0.00 -> 196.1 mm, vias 0 -> 5
- net 3V3: track 0.00 -> 192.9 mm
- net SDA: track 0.00 -> 190.7 mm, vias 0 -> 4
- net +5V: track 0.00 -> 189.9 mm, vias 0 -> 1
- net SCL: track 0.00 -> 185.0 mm, vias 0 -> 1
- net 5V: track 0.00 -> 173.6 mm, vias 0 -> 2
- net MOSI: track 0.00 -> 151.9 mm
- net SS: track 0.00 -> 138.5 mm, vias 0 -> 1
- net N$4: track 0.00 -> 109.7 mm
- net MISO: track 0.00 -> 79.4 mm
- net RX0: track 0.00 -> 76.7 mm
- net TX1: track 0.00 -> 59.0 mm
- net SCK: track 0.00 -> 51.7 mm
- net SBG_RX: track 0.00 -> 35.7 mm
- net SBG_TX: track 0.00 -> 35.2 mm
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
Commit message: final revisions
Parts:
- moved POWER_IN 6.77 mm to (17.2, 126.0), flipped to the bottom, turned to 90 degrees
Connections:
- removed net +5V: AIR_BRAKE.2, ARDUINO_NANO1.15, POWER_IN.1
- new net VIN: ARDUINO_NANO1.15
- net 3V3: now also U$7.VIN; no longer R_SCL.1, R_SDA.1
- net 5V: now also AIR_BRAKE.2, POWER_IN.1, R_SCL.1, R_SDA.1
Routing:
- net +5V: track 189.9 -> 0.00 mm, vias 1 -> 0
- net 5V: track 173.6 -> 271.1 mm
- net MOSI: track 151.9 -> 70.6 mm
- net SS: track 138.5 -> 68.8 mm, vias 1 -> 0
- net SDA: track 190.7 -> 122.9 mm, vias 4 -> 2
- net GND: track 196.1 -> 239.8 mm, vias 5 -> 1
- net SCK: track 51.7 -> 92.2 mm, vias 0 -> 1
- net 3V3: track 192.9 -> 177.7 mm, vias 0 -> 1
- net N$4: track 109.7 -> 122.1 mm
- net SCL: track 185.0 -> 188.0 mm, vias 1 -> 2
- net MISO: track 79.4 -> 76.5 mm
- net TX: track 24.4 -> 23.2 mm
- net RX0: track 76.7 -> 76.5 mm, vias 0 -> 2
Other:
- outline, holes or cut-outs redrawn
