File: Powerboard/Powerboard.brd (EAGLE design)
At the start: 87.5 x 150 mm, 9 parts

Commit message: refactor
Parts:
- added J3: (no value), SparkFun-Connectors:SCREWTERMINAL-3.5MM-2
Routing:
- net VIN: track 4.75 -> 7.50 mm
Changed lines of the file:
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@@
 <text x="56.313" y="136.9434" size="1.016" layer="21" font="vector" ratio="15" rot="R180">VOUT</text>
 <text x="56.313" y="131.8634" size="1.016" layer="21" font="vector" ratio="15" rot="R180">TRIM</text>
-<hole x="9.75" y="140" drill="5.5"/>
-<hole x="9.75" y="10" drill="5.5"/>
-<hole x="77.75" y="10" drill="5.5"/>
-<hole x="77.75" y="140" drill="5.5"/>
+<hole x="9.75" y="140" drill="6.6"/>
+<hole x="9.75" y="10" drill="6.6"/>
+<hole x="77.75" y="10" drill="6.6"/>
+<hole x="77.75" y="140" drill="6.6"/>
 <dimension x1="77.75" y1="142.75" x2="77.75" y2="137.25" x3="97" y3="140" textsize="1.778" layer="47" dtype="diameter"/>
 <dimension x1="78" y1="140" x2="10" y2="140" x3="44" y3="169" textsize="1.778" layer="47" dtype="diameter"/>
@@
 <text x="70.5" y="125.5" size="1.778" layer="48">Power Board</text>
 <text x="74.5" y="122.5" size="1.778" layer="48">v1.0</text>
-<circle x="9.75" y="140" radius="4.125" width="0" layer="39"/>
-<circle x="77.75" y="140" radius="4.125" width="0" layer="39"/>
-<circle x="77.75" y="10" radius="4.125" width="0" layer="39"/>
-<circle x="9.75" y="10" radius="4.125" width="0" layer="39"/>
+<circle x="9.75" y="140" radius="5.125" width="0" layer="39"/>
+<circle x="77.75" y="140" radius="5.125" width="0" layer="39"/>
+<circle x="77.75" y="10" radius="5.125" width="0" layer="39"/>
+<circle x="9.75" y="10" radius="5.125" width="0" layer="39"/>
+<wire x1="17.25" y1="115.25" x2="51.25" y2="115.25" width="0.2032" layer="51"/>
+<wire x1="51.25" y1="115.25" x2="51.25" y2="10.25" width="0.2032" layer="51"/>
+<wire x1="51.25" y1="10.25" x2="17.25" y2="10.25" width="0.2032" layer="51"/>
+<wire x1="17.25" y1="10.25" x2="17.25" y2="115.25" width="0.2032" layer="51"/>
 </plain>
 <attributes>
@@
 <attribute name="VALUE" x="20.802" y="134.811" size="0.6096" layer="27" font="vector" ratio="20" rot="R180"/>
 </element>
+<element name="J3" library="SparkFun-Connectors" package="SCREWTERMINAL-3.5MM-2" value="" x="4.75" y="126.75" smashed="yes">
+<attribute name="NAME" x="3.48" y="129.29" size="0.6096" layer="25" font="vector" ratio="20"/>
+<attribute name="PROD_ID" value="CONN-08399" x="4.75" y="126.75" size="1.778" layer="27" display="off"/>
+<attribute name="VALUE" x="3.48" y="128.02" size="0.6096" layer="27" font="vector" ratio="20"/>
+</element>
 </elements>
 <signals>
@@
 <vertex x="14" y="121"/>
 </polygon>
-<wire x1="17.5" y1="123" x2="22.25" y2="123" width="3.75" layer="1"/>
+<wire x1="17.5" y1="123" x2="15.75" y2="123" width="3.75" layer="1"/>
+<wire x1="17.5" y1="123" x2="22.75" y2="123" width="4" layer="1"/>
+<wire x1="22.75" y1="123" x2="23.25" y2="123" width="0.1524" layer="1"/>
 </signal>
 <signal name="VOUT">

Commit message: wip
Parts:
- moved OUT1 117.5 mm to (55.0, 13.8)
- moved U$2 117.5 mm to (32.1, 27.8)
- moved U$7 117.5 mm to (55.0, 27.8)
- moved R_TRIM 117.5 mm to (46.2, 14.5)
- moved U$6 117.5 mm to (32.1, 4.94)
- moved U$8 117.5 mm to (55.0, 4.94)
- moved IN1 117.5 mm to (32.1, 21.4)
- moved J2 105.5 mm to (20.2, 17.5)
- moved J3 105.5 mm to (7.50, 21.2)
- moved J1 14.9 mm to (79.5, 126.8)
Routing:
- net GND: track 18.8 -> 0.00 mm
- net VIN: track 7.50 -> 0.00 mm
- removed copper zone on layer 1, net GND
- removed copper zone on layer 1, net TRIM
- removed copper zone on layer 1, net VIN
- removed copper zone on layer 1, net VOUT

Commit message: powerboard layout
Parts:
- removed J1, J3: (no value), SparkFun-Connectors:SCREWTERMINAL-3.5MM-2
- removed J2: (no value), SparkFun-Connectors:DEANS
- added DEANS: (no value), SparkFun-Connectors:DEANS
- added SWITCH, TERMINAL_BLOCK, TO_MOTHERBOARD: (no value), SparkFun-Connectors:SCREWTERMINAL-3.5MM-2
Connections:
- new net N$1: DEANS.+, SWITCH.2, TERMINAL_BLOCK.2
- net GND: now also DEANS.-, TERMINAL_BLOCK.1, TO_MOTHERBOARD.2; no longer J1.2, J2.-
- net VIN: now also SWITCH.1; no longer J2.+
- net VOUT: now also TO_MOTHERBOARD.1; no longer J1.1
Changed lines of the file:
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@@
 <setting verticaltext="up"/>
 </settings>
-<grid distance="1" unitdist="mil" unit="mil" style="dots" multiple="1" display="yes" altdistance="5" altunitdist="mil" altunit="mil"/>
+<grid distance="1" unitdist="mm" unit="mm" style="dots" multiple="1" display="yes" altdistance="5" altunitdist="mil" altunit="mil"/>
 <layers>
 <layer number="1" name="Top" color="4" fill="1" visible="yes" active="yes"/>
@@
 <dimension x1="26" y1="150" x2="26" y2="0" x3="-15" y3="75" textsize="1.778" layer="47"/>
 <dimension x1="0" y1="49.5" x2="87.5" y2="49.5" x3="43.75" y3="-7" textsize="1.778" layer="47"/>
-<text x="84" y="125.75" size="1.778" layer="47">+</text>
-<text x="84" y="129.75" size="1.778" layer="47">-</text>
-<text x="67" y="59" size="1.778" layer="48">uORocketry </text>
-<text x="66.25" y="56" size="1.778" layer="48">Power Board</text>
-<text x="70" y="52.75" size="1.778" layer="48">v1.0</text>
+<text x="84" y="79.75" size="1.778" layer="47">+</text>
+<text x="84" y="83.75" size="1.778" layer="47">-</text>
+<text x="6" y="99" size="1.778" layer="48">uORocketry </text>
+<text x="6.25" y="95" size="1.778" layer="48">Power Board</text>
+<text x="12" y="91.75" size="1.778" layer="48">v1.0</text>
 <circle x="9.75" y="140" radius="5.125" width="0" layer="39"/>
 <circle x="77.75" y="140" radius="5.125" width="0" layer="39"/>
 <circle x="77.75" y="10" radius="5.125" width="0" layer="39"/>
 <circle x="9.75" y="10" radius="5.125" width="0" layer="39"/>
-<wire x1="25" y1="148.25" x2="59" y2="148.25" width="0.2032" layer="51"/>
-<wire x1="59" y1="148.25" x2="59" y2="43.25" width="0.2032" layer="102"/>
-<wire x1="59" y1="43.25" x2="25" y2="43.25" width="0.2032" layer="51"/>
-<wire x1="25" y1="43.25" x2="25" y2="148.25" width="0.2032" layer="51"/>
+<hole x="15" y="114.77" drill="12"/>
+<wire x1="8" y1="36" x2="8" y2="71" width="0.1524" layer="51"/>
+<wire x1="8" y1="71" x2="78" y2="71" width="0.1524" layer="51"/>
+<wire x1="78" y1="71" x2="78" y2="36" width="0.1524" layer="51"/>
+<wire x1="78" y1="36" x2="8" y2="36" width="0.1524" layer="51"/>
+<hole x="43" y="34" drill="3.4"/>
+<hole x="81" y="34" drill="3.4"/>
+<hole x="5" y="33" drill="3.4"/>
+<hole x="21" y="74" drill="3.4"/>
+<hole x="61" y="74" drill="3.4"/>
+<hole x="62" y="33" drill="3.4"/>
+<hole x="20" y="33" drill="3.4"/>
+<hole x="31.38" y="133.85" drill="4"/>
+<hole x="70.38" y="133.85" drill="4"/>
+<hole x="31.38" y="94.85" drill="4"/>
+<hole x="70.38" y="94.85" drill="4"/>
+<hole x="13" y="21" drill="3.4"/>
+<hole x="26" y="21" drill="3.4"/>
 </plain>
 <attributes>
@@
 <attribute name="VALUE" x="44.345" y="15.135" size="1.27" layer="27" rot="R270"/>
 </element>
-<element name="J1" library="SparkFun-Connectors" package="SCREWTERMINAL-3.5MM-2" value="" x="79.5" y="126.75" smashed="yes" rot="R90">
-<attribute name="NAME" x="76.96" y="125.48" size="0.6096" layer="25" font="vector" ratio="20" rot="R90"/>
-<attribute name="PROD_ID" value="CONN-08399" x="79.5" y="126.75" size="1.778" layer="27" rot="R90" display="off"/>
-<attribute name="VALUE" x="78.23" y="125.48" size="0.6096" layer="27" font="vector" ratio="20" rot="R90"/>
-</element>
-<element name="J2" library="SparkFun-Connectors" package="DEANS" value="" x="20.25" y="17.5" smashed="yes" rot="R180">
-<attribute name="NAME" x="24.06" y="14.96" size="0.6096" layer="25" font="vector" ratio="20" rot="R180"/>
-<attribute name="SF_ID" value="PRT-11864" x="20.25" y="17.5" size="1.778" layer="27" rot="R180" display="off"/>
-<attribute name="VALUE" x="23.552" y="29.311" size="0.6096" layer="27" font="vector" ratio="20" rot="R180"/>
-</element>
-<element name="J3" library="SparkFun-Connectors" package="SCREWTERMINAL-3.5MM-2" value="" x="7.5" y="21.25" smashed="yes">
-<attribute name="NAME" x="6.23" y="23.79" size="0.6096" layer="25" font="vector" ratio="20"/>
-<attribute name="PROD_ID" value="CONN-08399" x="7.5" y="21.25" size="1.778" layer="27" display="off"/>
-<attribute name="VALUE" x="6.23" y="22.52" size="0.6096" layer="27" font="vector" ratio="20"/>
+<element name="TO_MOTHERBOARD" library="SparkFun-Connectors" package="SCREWTERMINAL-3.5MM-2" value="" x="79.5" y="80.75" smashed="yes" rot="R90">
+<attribute name="NAME" x="76.96" y="79.48" size="0.6096" layer="25" font="vector" ratio="20" rot="R90"/>
+<attribute name="PROD_ID" value="CONN-08399" x="79.5" y="80.75" size="1.778" layer="27" rot="R90" display="off"/>
+<attribute name="VALUE" x="78.23" y="79.48" size="0.6096" layer="27" font="vector" ratio="20" rot="R90"/>
+</element>
+<element name="DEANS" library="SparkFun-Connectors" package="DEANS" value="" x="19.25" y="17.5" smashed="yes" rot="R180">
+<attribute name="NAME" x="23.06" y="14.96" size="0.6096" layer="25" font="vector" ratio="20" rot="R180"/>
+<attribute name="SF_ID" value="PRT-11864" x="19.25" y="17.5" size="1.778" layer="27" rot="R180" display="off"/>
+<attribute name="VALUE" x="22.552" y="29.311" size="0.6096" layer="27" font="vector" ratio="20" rot="R180"/>
+</element>
+<element name="TERMINAL_BLOCK" library="SparkFun-Connectors" package="SCREWTERMINAL-3.5MM-2" value="" x="4.5" y="22.25" smashed="yes">
+<attribute name="NAME" x="3.23" y="24.79" size="0.6096" layer="25" font="vector" ratio="20"/>
+<attribute name="PROD_ID" value="CONN-08399" x="4.5" y="22.25" size="1.778" layer="27" display="off"/>
+<attribute name="VALUE" x="3.23" y="23.52" size="0.6096" layer="27" font="vector" ratio="20"/>
+</element>
+<element name="SWITCH" library="SparkFun-Connectors" package="SCREWTERMINAL-3.5MM-2" value="" x="17" y="86" smashed="yes" rot="R180">
+<attribute name="NAME" x="18.27" y="83.46" size="0.6096" layer="25" font="vector" ratio="20" rot="R180"/>
+<attribute name="PROD_ID" value="CONN-08399" x="17" y="86" size="1.778" layer="27" rot="R180" display="off"/>
+<attribute name="VALUE" x="18.27" y="84.73" size="0.6096" layer="27" font="vector" ratio="20" rot="R180"/>
 </element>
 </elements>
@@
 <contactref element="OUT1" pad="2"/>
 <contactref element="R_TRIM" pad="1"/>
-<contactref element="J2" pad="-"/>
-<contactref element="J1" pad="2"/>
+<contactref element="DEANS" pad="-"/>
+<contactref element="TO_MOTHERBOARD" pad="2"/>
+<contactref element="TERMINAL_BLOCK" pad="1"/>
+<wire x1="54.96" y1="16.37" x2="79.5" y2="84.25" width="0" layer="19" extent="1-1"/>
+<wire x1="46.25" y1="15.35" x2="54.96" y2="16.37" width="0" layer="19" extent="1-1"/>
+<wire x1="32.1" y1="13.83" x2="46.25" y2="15.35" width="0" layer="19" extent="1-1"/>
+<wire x1="18.5134" y1="24.4215" x2="32.1" y2="13.83" width="0" layer="19" extent="1-1"/>
+<wire x1="4.5" y1="22.25" x2="18.5134" y2="24.4215" width="0" layer="19" extent="1-1"/>
 </signal>
 <signal name="SEQ">
@@
 <contactref element="OUT1" pad="1"/>
 <contactref element="R_TRIM" pad="2"/>
+<wire x1="46.25" y1="13.65" x2="54.96" y2="13.83" width="0" layer="19" extent="1-1"/>
 </signal>
 <signal name="ON/OFF">
@@
 <signal name="VIN">
 <contactref element="IN1" pad="5"/>
-<contactref element="J2" pad="+"/>
+<contactref element="SWITCH" pad="1"/>
+<wire x1="17" y1="86" x2="32.1" y2="11.29" width="0" layer="19" extent="1-1"/>
 </signal>
 <signal name="VOUT">
 <contactref element="OUT1" pad="3"/>
-<contactref element="J1" pad="1"/>
+<contactref element="TO_MOTHERBOARD" pad="1"/>
+<wire x1="54.96" y1="18.91" x2="79.5" y2="80.75" width="0" layer="19" extent="1-1"/>
+</signal>
+<signal name="N$1">
+<contactref element="DEANS" pad="+"/>
+<contactref element="TERMINAL_BLOCK" pad="2"/>
+<contactref element="SWITCH" pad="2"/>
+<wire x1="8" y1="22.25" x2="19.25" y2="17.5" width="0" layer="19" extent="1-1"/>
+<wire x1="13.5" y1="86" x2="8" y2="22.25" width="0" layer="19" extent="1-1"/>
 </signal>
 </signals>

Commit message: routing
Routing:
- net GND: track 0.00 -> 150.2 mm
- net VIN: track 0.00 -> 85.2 mm
- net N$1: track 0.00 -> 79.2 mm
- net VOUT: track 0.00 -> 72.3 mm
- net TRIM: track 0.00 -> 8.78 mm
Changed lines of the file:
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@@
 <contactref element="TO_MOTHERBOARD" pad="2"/>
 <contactref element="TERMINAL_BLOCK" pad="1"/>
-<wire x1="54.96" y1="16.37" x2="79.5" y2="84.25" width="0" layer="19" extent="1-1"/>
-<wire x1="46.25" y1="15.35" x2="54.96" y2="16.37" width="0" layer="19" extent="1-1"/>
-<wire x1="32.1" y1="13.83" x2="46.25" y2="15.35" width="0" layer="19" extent="1-1"/>
-<wire x1="18.5134" y1="24.4215" x2="32.1" y2="13.83" width="0" layer="19" extent="1-1"/>
-<wire x1="4.5" y1="22.25" x2="18.5134" y2="24.4215" width="0" layer="19" extent="1-1"/>
+<wire x1="42.672" y1="14.224" x2="32.004" y2="14.224" width="1.778" layer="1"/>
+<wire x1="12.446" y1="14.224" x2="5.334" y2="21.336" width="1.778" layer="1"/>
+<wire x1="32.004" y1="14.224" x2="12.446" y2="14.224" width="1.778" layer="1"/>
+<wire x1="5.334" y1="21.336" x2="4.5" y2="22.25" width="1.778" layer="1"/>
+<wire x1="32.004" y1="14.224" x2="32.1" y2="13.83" width="1.778" layer="1"/>
+<wire x1="78.232" y1="83.566" x2="80.01" y2="83.566" width="1.778" layer="1"/>
+<wire x1="58.674" y1="64.008" x2="78.232" y2="83.566" width="1.778" layer="1"/>
+<wire x1="58.674" y1="19.558" x2="58.674" y2="64.008" width="1.778" layer="1"/>
+<wire x1="55.118" y1="16.002" x2="58.674" y2="19.558" width="1.778" layer="1"/>
+<wire x1="80.01" y1="83.566" x2="79.5" y2="84.25" width="1.778" layer="1"/>
+<wire x1="55.118" y1="16.002" x2="54.96" y2="16.37" width="1.778" layer="1"/>
+<wire x1="18.5134" y1="24.4215" x2="6.6715" y2="24.4215" width="1.778" layer="16"/>
+<wire x1="6.6715" y1="24.4215" x2="4.5" y2="22.25" width="1.778" layer="16"/>
+<wire x1="46.25" y1="15.35" x2="46.902" y2="16.002" width="1.27" layer="1"/>
+<wire x1="46.902" y1="16.002" x2="55.118" y2="16.002" width="1.778" layer="1"/>
+<wire x1="46.25" y1="15.35" x2="43.798" y2="15.35" width="1.27" layer="1"/>
+<wire x1="43.798" y1="15.35" x2="42.672" y2="14.224" width="1.778" layer="1"/>
 </signal>
 <signal name="SEQ">
@@
 <contactref element="OUT1" pad="1"/>
 <contactref element="R_TRIM" pad="2"/>
-<wire x1="46.25" y1="13.65" x2="54.96" y2="13.83" width="0" layer="19" extent="1-1"/>
+<wire x1="46.25" y1="13.65" x2="54.78" y2="13.65" width="1.27" layer="1"/>
+<wire x1="54.78" y1="13.65" x2="54.96" y2="13.83" width="1.778" layer="1"/>
 </signal>
 <signal name="ON/OFF">
@@
 <contactref element="IN1" pad="5"/>
 <contactref element="SWITCH" pad="1"/>
-<wire x1="17" y1="86" x2="32.1" y2="11.29" width="0" layer="19" extent="1-1"/>
+<wire x1="35.56" y1="14.224" x2="32.004" y2="10.668" width="1.778" layer="16"/>
+<wire x1="35.56" y1="67.564" x2="35.56" y2="14.224" width="1.778" layer="16"/>
+<wire x1="17.78" y1="85.344" x2="35.56" y2="67.564" width="1.778" layer="16"/>
+<wire x1="32.004" y1="10.668" x2="32.1" y2="11.29" width="1.778" layer="16"/>
+<wire x1="17.78" y1="85.344" x2="17" y2="86" width="1.778" layer="16"/>
 </signal>
 <signal name="VOUT">
 <contactref element="OUT1" pad="3"/>
 <contactref element="TO_MOTHERBOARD" pad="1"/>
-<wire x1="54.96" y1="18.91" x2="79.5" y2="80.75" width="0" layer="19" extent="1-1"/>
+<wire x1="80.01" y1="44.45" x2="55.118" y2="19.558" width="1.778" layer="16"/>
+<wire x1="80.01" y1="80.01" x2="80.01" y2="44.45" width="1.778" layer="16"/>
+<wire x1="55.118" y1="19.558" x2="54.96" y2="18.91" width="1.778" layer="16"/>
+<wire x1="80.01" y1="80.01" x2="79.5" y2="80.75" width="1.778" layer="16"/>
 </signal>
 <signal name="N$1">
@@
 <contactref element="TERMINAL_BLOCK" pad="2"/>
 <contactref element="SWITCH" pad="2"/>
-<wire x1="8" y1="22.25" x2="19.25" y2="17.5" width="0" layer="19" extent="1-1"/>
-<wire x1="13.5" y1="86" x2="8" y2="22.25" width="0" layer="19" extent="1-1"/>
+<wire x1="13.5" y1="86" x2="13.5" y2="27.75" width="1.778" layer="1"/>
+<wire x1="13.5" y1="27.75" x2="8" y2="22.25" width="1.778" layer="1"/>
+<wire x1="19.25" y1="17.5" x2="12.75" y2="17.5" width="1.778" layer="1"/>
+<wire x1="12.75" y1="17.5" x2="8" y2="22.25" width="1.778" layer="1"/>
 </signal>
 </signals>

Commit message: review1
Parts:
- moved TERMINAL_BLOCK 22.5 mm to (22.5, 8.75), turned to 180 degrees
- moved TO_MOTHERBOARD 7.00 mm to (72.5, 80.8)
Routing:
- net N$1: track 79.2 -> 162.6 mm
- net GND: track 150.2 -> 230.4 mm
- net VOUT: track 72.3 -> 74.5 mm
Changed lines of the file:
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@@
 <dimension x1="26" y1="150" x2="26" y2="0" x3="-15" y3="75" textsize="1.778" layer="47"/>
 <dimension x1="0" y1="49.5" x2="87.5" y2="49.5" x3="43.75" y3="-7" textsize="1.778" layer="47"/>
-<text x="84" y="79.75" size="1.778" layer="47">+</text>
-<text x="84" y="83.75" size="1.778" layer="47">-</text>
+<text x="77" y="79.75" size="1.778" layer="47">+</text>
+<text x="77" y="83.75" size="1.778" layer="47">-</text>
 <text x="6" y="99" size="1.778" layer="48">uORocketry </text>
 <text x="6.25" y="95" size="1.778" layer="48">Power Board</text>
@@
 <attribute name="VALUE" x="44.345" y="15.135" size="1.27" layer="27" rot="R270"/>
 </element>
-<element name="TO_MOTHERBOARD" library="SparkFun-Connectors" package="SCREWTERMINAL-3.5MM-2" value="" x="79.5" y="80.75" smashed="yes" rot="R90">
-<attribute name="NAME" x="76.96" y="79.48" size="0.6096" layer="25" font="vector" ratio="20" rot="R90"/>
-<attribute name="PROD_ID" value="CONN-08399" x="79.5" y="80.75" size="1.778" layer="27" rot="R90" display="off"/>
-<attribute name="VALUE" x="78.23" y="79.48" size="0.6096" layer="27" font="vector" ratio="20" rot="R90"/>
+<element name="TO_MOTHERBOARD" library="SparkFun-Connectors" package="SCREWTERMINAL-3.5MM-2" value="" x="72.5" y="80.75" smashed="yes" rot="R90">
+<attribute name="NAME" x="69.96" y="79.48" size="0.6096" layer="25" font="vector" ratio="20" rot="R90"/>
+<attribute name="PROD_ID" value="CONN-08399" x="72.5" y="80.75" size="1.778" layer="27" rot="R90" display="off"/>
+<attribute name="VALUE" x="71.23" y="79.48" size="0.6096" layer="27" font="vector" ratio="20" rot="R90"/>
 </element>
 <element name="DEANS" library="SparkFun-Connectors" package="DEANS" value="" x="19.25" y="17.5" smashed="yes" rot="R180">
@@
 <attribute name="VALUE" x="22.552" y="29.311" size="0.6096" layer="27" font="vector" ratio="20" rot="R180"/>
 </element>
-<element name="TERMINAL_BLOCK" library="SparkFun-Connectors" package="SCREWTERMINAL-3.5MM-2" value="" x="4.5" y="22.25" smashed="yes">
-<attribute name="NAME" x="3.23" y="24.79" size="0.6096" layer="25" font="vector" ratio="20"/>
-<attribute name="PROD_ID" value="CONN-08399" x="4.5" y="22.25" size="1.778" layer="27" display="off"/>
-<attribute name="VALUE" x="3.23" y="23.52" size="0.6096" layer="27" font="vector" ratio="20"/>
+<element name="TERMINAL_BLOCK" library="SparkFun-Connectors" package="SCREWTERMINAL-3.5MM-2" value="" x="22.5" y="8.75" smashed="yes" rot="R180">
+<attribute name="NAME" x="23.77" y="6.21" size="0.6096" layer="25" font="vector" ratio="20" rot="R180"/>
+<attribute name="PROD_ID" value="CONN-08399" x="22.5" y="8.75" size="1.778" layer="27" rot="R180" display="off"/>
+<attribute name="VALUE" x="23.77" y="7.48" size="0.6096" layer="27" font="vector" ratio="20" rot="R180"/>
 </element>
 <element name="SWITCH" library="SparkFun-Connectors" package="SCREWTERMINAL-3.5MM-2" value="" x="17" y="86" smashed="yes" rot="R180">
@@
 <contactref element="TERMINAL_BLOCK" pad="1"/>
 <wire x1="42.672" y1="14.224" x2="32.004" y2="14.224" width="1.778" layer="1"/>
-<wire x1="12.446" y1="14.224" x2="5.334" y2="21.336" width="1.778" layer="1"/>
-<wire x1="32.004" y1="14.224" x2="12.446" y2="14.224" width="1.778" layer="1"/>
-<wire x1="5.334" y1="21.336" x2="4.5" y2="22.25" width="1.778" layer="1"/>
+<wire x1="22.5" y1="8.75" x2="54.84220625" y2="15.35" width="1.778" layer="1"/>
+<wire x1="46.25" y1="15.35" x2="54.84220625" y2="15.35" width="1.778" layer="1"/>
 <wire x1="32.004" y1="14.224" x2="32.1" y2="13.83" width="1.778" layer="1"/>
-<wire x1="78.232" y1="83.566" x2="80.01" y2="83.566" width="1.778" layer="1"/>
-<wire x1="58.674" y1="64.008" x2="78.232" y2="83.566" width="1.778" layer="1"/>
+<wire x1="58.674" y1="64.008" x2="75.240503125" y2="80.574503125" width="1.778" layer="1"/>
 <wire x1="58.674" y1="19.558" x2="58.674" y2="64.008" width="1.778" layer="1"/>
 <wire x1="55.118" y1="16.002" x2="58.674" y2="19.558" width="1.778" layer="1"/>
-<wire x1="80.01" y1="83.566" x2="79.5" y2="84.25" width="1.778" layer="1"/>
+<wire x1="75.240503125" y1="80.574503125" x2="72.5" y2="84.25" width="1.778" layer="1"/>
 <wire x1="55.118" y1="16.002" x2="54.96" y2="16.37" width="1.778" layer="1"/>
-<wire x1="18.5134" y1="24.4215" x2="6.6715" y2="24.4215" width="1.778" layer="16"/>
-<wire x1="6.6715" y1="24.4215" x2="4.5" y2="22.25" width="1.778" layer="16"/>
+<wire x1="22.5" y1="8.75" x2="62.3285" y2="24.4215" width="1.778" layer="16"/>
+<wire x1="18.5134" y1="24.4215" x2="62.3285" y2="24.4215" width="1.778" layer="16"/>
 <wire x1="46.25" y1="15.35" x2="46.902" y2="16.002" width="1.27" layer="1"/>
 <wire x1="46.902" y1="16.002" x2="55.118" y2="16.002" width="1.778" layer="1"/>
@@
 <contactref element="TO_MOTHERBOARD" pad="1"/>
 <wire x1="80.01" y1="44.45" x2="55.118" y2="19.558" width="1.778" layer="16"/>
-<wire x1="80.01" y1="80.01" x2="80.01" y2="44.45" width="1.778" layer="16"/>
+<wire x1="80.01" y1="69.8531375" x2="80.01" y2="44.45" width="1.778" layer="16"/>
 <wire x1="55.118" y1="19.558" x2="54.96" y2="18.91" width="1.778" layer="16"/>
-<wire x1="80.01" y1="80.01" x2="79.5" y2="80.75" width="1.778" layer="16"/>
+<wire x1="80.01" y1="69.8531375" x2="72.5" y2="80.75" width="1.778" layer="16"/>
 </signal>
 <signal name="N$1">
@@
 <contactref element="TERMINAL_BLOCK" pad="2"/>
 <contactref element="SWITCH" pad="2"/>
-<wire x1="13.5" y1="86" x2="13.5" y2="27.75" width="1.778" layer="1"/>
-<wire x1="13.5" y1="27.75" x2="8" y2="22.25" width="1.778" layer="1"/>
-<wire x1="19.25" y1="17.5" x2="12.75" y2="17.5" width="1.778" layer="1"/>
-<wire x1="12.75" y1="17.5" x2="8" y2="22.25" width="1.778" layer="1"/>
+<wire x1="13.5" y1="86" x2="13.5" y2="76.75" width="1.778" layer="1"/>
+<wire x1="13.5" y1="76.75" x2="19" y2="8.75" width="1.778" layer="1"/>
+<wire x1="19" y1="8.75" x2="61.25" y2="17.5" width="1.778" layer="1"/>
+<wire x1="19.25" y1="17.5" x2="61.25" y2="17.5" width="1.778" layer="1"/>
 </signal>
 </signals>

Commit message: layout r2
Parts:
- removed TERMINAL_BLOCK: (no value), SparkFun-Connectors:SCREWTERMINAL-3.5MM-2
- added BATTERY_TERMINAL_BLOCK: (no value), SparkFun-Connectors:SCREWTERMINAL-3.5MM-2
- moved DEANS 51.9 mm to (41.2, 64.5), flipped to the bottom
- moved IN1 28.1 mm to (30.1, 49.5)
- moved OUT1 28.1 mm to (53.0, 41.8)
- moved R_TRIM 28.1 mm to (44.2, 42.5)
- moved U$2 28.1 mm to (30.1, 55.8)
- moved U$6 28.1 mm to (30.1, 32.9)
- moved U$7 28.1 mm to (53.0, 55.8)
- moved U$8 28.1 mm to (53.0, 32.9)
- moved TO_MOTHERBOARD 4.00 mm to (68.5, 80.8)
- moved SWITCH 1.00 mm to (18.0, 86.0), flipped to the bottom
Connections:
- net GND: now also BATTERY_TERMINAL_BLOCK.1, TO_MOTHERBOARD.1; no longer TERMINAL_BLOCK.1, TO_MOTHERBOARD.2
- net N$1: now also BATTERY_TERMINAL_BLOCK.2; no longer TERMINAL_BLOCK.2
- net VOUT: now also TO_MOTHERBOARD.2; no longer TO_MOTHERBOARD.1
Routing:
- net GND: track 230.4 -> 0.00 mm
- net N$1: track 162.6 -> 0.00 mm
- net VIN: track 85.2 -> 0.00 mm
- net VOUT: track 74.5 -> 0.00 mm
- net TRIM: track 8.78 -> 0.00 mm
