File: Powerboard/Powerboard.brd (EAGLE design)
At the start: 87.5 x 150 mm, 11 parts

Commit message: route powerboard r2
Routing:
- net GND: track 0.00 -> 117.2 mm
- net VIN: track 0.00 -> 51.8 mm
- net VOUT: track 0.00 -> 43.8 mm
- net N$1: track 0.00 -> 36.3 mm
- net TRIM: track 0.00 -> 8.78 mm
Changed lines of the file:
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@@
 <contactref element="BATTERY_TERMINAL_BLOCK" pad="1"/>
 <contactref element="TO_MOTHERBOARD" pad="1"/>
-<wire x1="41.9866" y1="71.4215" x2="68.5" y2="80.75" width="0" layer="19" extent="1-1"/>
-<wire x1="23.5" y1="67.75" x2="41.9866" y2="71.4215" width="0" layer="19" extent="1-1"/>
-<wire x1="30.1" y1="41.83" x2="23.5" y2="67.75" width="0" layer="19" extent="1-1"/>
-<wire x1="44.25" y1="43.35" x2="30.1" y2="41.83" width="0" layer="19" extent="1-1"/>
-<wire x1="52.96" y1="44.37" x2="44.25" y2="43.35" width="0" layer="19" extent="1-1"/>
+<wire x1="52.9562" y1="44.3738" x2="45.6251625" y2="44.3738" width="1.016" layer="1"/>
+<wire x1="52.9562" y1="44.3738" x2="52.96" y2="44.37" width="1.016" layer="1"/>
+<wire x1="44.704" y1="43.688" x2="34.544" y2="43.688" width="1.016" layer="1"/>
+<wire x1="34.544" y1="43.688" x2="33.705471875" y2="41.83" width="1.016" layer="1"/>
+<wire x1="33.705471875" y1="41.83" x2="30.1" y2="41.83" width="1.016" layer="1"/>
+<wire x1="45.6251625" y1="44.3738" x2="44.704" y2="43.688" width="1.016" layer="1"/>
+<wire x1="44.704" y1="43.688" x2="44.25" y2="43.35" width="1.016" layer="1"/>
+<wire x1="24.384" y1="46.736" x2="24.384" y2="67.056" width="1.016" layer="1"/>
+<wire x1="29.464" y1="41.656" x2="24.384" y2="46.736" width="1.016" layer="1"/>
+<wire x1="24.384" y1="67.056" x2="23.5" y2="67.75" width="1.016" layer="1"/>
+<wire x1="29.464" y1="41.656" x2="30.1" y2="41.83" width="1.016" layer="1"/>
+<wire x1="68.072" y1="58.928" x2="68.072" y2="80.264" width="1.016" layer="1"/>
+<wire x1="53.848" y1="44.704" x2="68.072" y2="58.928" width="1.016" layer="1"/>
+<wire x1="68.072" y1="80.264" x2="68.5" y2="80.75" width="1.016" layer="1"/>
+<wire x1="53.848" y1="44.704" x2="52.96" y2="44.37" width="1.016" layer="1"/>
+<wire x1="41.9866" y1="71.4215" x2="27.1715" y2="71.4215" width="1.016" layer="16"/>
+<wire x1="27.1715" y1="71.4215" x2="23.5" y2="67.75" width="1.016" layer="16"/>
 </signal>
 <signal name="SEQ">
@@
 <contactref element="OUT1" pad="1"/>
 <contactref element="R_TRIM" pad="2"/>
-<wire x1="44.25" y1="41.65" x2="52.96" y2="41.83" width="0" layer="19" extent="1-1"/>
+<wire x1="44.25" y1="41.65" x2="52.78" y2="41.65" width="1.016" layer="1"/>
+<wire x1="52.78" y1="41.65" x2="52.96" y2="41.83" width="1.016" layer="1"/>
 </signal>
 <signal name="ON/OFF">
@@
 <contactref element="IN1" pad="5"/>
 <contactref element="SWITCH" pad="1"/>
-<wire x1="30.1" y1="39.29" x2="18" y2="86" width="0" layer="19" extent="1-1"/>
+<wire x1="18.288" y1="50.8" x2="29.464" y2="39.624" width="1.016" layer="16"/>
+<wire x1="18.288" y1="85.344" x2="18.288" y2="50.8" width="1.016" layer="16"/>
+<wire x1="29.464" y1="39.624" x2="30.1" y2="39.29" width="1.016" layer="16"/>
+<wire x1="18.288" y1="85.344" x2="18" y2="86" width="1.016" layer="16"/>
 </signal>
 <signal name="VOUT">
 <contactref element="OUT1" pad="3"/>
 <contactref element="TO_MOTHERBOARD" pad="2"/>
-<wire x1="52.96" y1="46.91" x2="68.5" y2="84.25" width="0" layer="19" extent="1-1"/>
+<wire x1="52.832" y1="50.8" x2="52.832" y2="47.752" width="1.016" layer="16"/>
+<wire x1="66.04" y1="64.008" x2="52.832" y2="50.8" width="1.016" layer="16"/>
+<wire x1="66.04" y1="81.28" x2="66.04" y2="64.008" width="1.016" layer="16"/>
+<wire x1="68.072" y1="83.312" x2="66.04" y2="81.28" width="1.016" layer="16"/>
+<wire x1="52.832" y1="47.752" x2="52.96" y2="46.91" width="1.016" layer="16"/>
+<wire x1="68.072" y1="83.312" x2="68.5" y2="84.25" width="1.016" layer="16"/>
 </signal>
 <signal name="N$1">
@@
 <contactref element="BATTERY_TERMINAL_BLOCK" pad="2"/>
 <contactref element="SWITCH" pad="2"/>
-<wire x1="41.25" y1="64.5" x2="21.5" y2="86" width="0" layer="19" extent="1-1"/>
-<wire x1="27" y1="67.75" x2="41.25" y2="64.5" width="0" layer="19" extent="1-1"/>
+<wire x1="26.416" y1="80.264" x2="26.416" y2="68.072" width="1.016" layer="1"/>
+<wire x1="21.336" y1="85.344" x2="26.416" y2="80.264" width="1.016" layer="1"/>
+<wire x1="26.416" y1="68.072" x2="27" y2="67.75" width="1.016" layer="1"/>
+<wire x1="21.336" y1="85.344" x2="21.5" y2="86" width="1.016" layer="1"/>
+<wire x1="41.25" y1="64.5" x2="30.25" y2="64.5" width="1.016" layer="1"/>
+<wire x1="30.25" y1="64.5" x2="27" y2="67.75" width="1.016" layer="1"/>
 </signal>
 </signals>
@@
 <mfgpreviewcolor name="substratecolor" color="0xFF786E46"/>
 </mfgpreviewcolors>
+<errors>
+</errors>
 </board>
 </drawing>

Commit message: final revisions
Parts:
- moved DEANS 50.6 mm to (68.8, 107.0)
- moved BATTERY_TERMINAL_BLOCK 5.50 mm to (18.0, 67.6)
- moved SWITCH 5.10 mm to (17.9, 80.9)
- moved TO_MOTHERBOARD 0.39 mm to (68.8, 81.0), flipped to the bottom, turned to 270 degrees
Connections:
- removed net N$1: BATTERY_TERMINAL_BLOCK.2, DEANS.+, SWITCH.2
- net ON/OFF: now also BATTERY_TERMINAL_BLOCK.2, DEANS.+, SWITCH.2
Routing:
- net ON/OFF: track 0.00 -> 102.9 mm
- net N$1: track 36.3 -> 0.00 mm
- net GND: track 117.2 -> 151.0 mm
- net VOUT: track 43.8 -> 37.4 mm
- net VIN: track 51.8 -> 46.7 mm
